File: hardware/satellite-board/satellite-board.kicad_sch (KiCad schematic)
At the start: 4 parts, among them U1 LORA1262-915TCXO, U2 XC6220B331MR, U3 ESP32-C6-DEVKITC-1-N8, U4 MAX3485

Commit message: wait more changes
Parts:
- added AE1: Antenna, symbol Device:Antenna
- added C1: 4.7 uF, symbol Device:C
- added C2: 10 uF, symbol Device:C
- added C3: 10uF, symbol Device:C
- added C4: 100nF, symbol Device:C
- added J1: MTJ-88ARX1-FSM-LG, MTJ-88ARX1-FSM-LG:ADAMTECH_MTJ-88ARX1-FSM-LG, symbol MTJ-88ARX1-FSM-LG:MTJ-88ARX1-FSM-LG
- added R1, R2: 150, symbol Device:R
Connections:
- net +3V3: now reaches U4.2 (~{RE})
- net +3V3: now also U1.13 (VCC), U2.5 (VOUT), U3.J1_1 (ESP_3V3), U4.8 (VCC), C1.1, C3.1, C4.1
- net RS_EN: now reaches U4.3 (DE)
- net RS_TX: now reaches U4.4 (DI)
- net GND: now reaches U4.5 (GND)
- net GND: now also U1.1 (GND), U1.10 (GND), U1.8 (GND), U2.2 (GND), U3.J1_15 (GND_J1_15), U3.J3_1 (GND_J3_1), U3.J3_12 (GND_J3_12), U3.J3_15 (GND_J3_15), C1.2, C2.2, C3.2, C4.2, J1.11, J1.7, J1.8, J1.9, J1.SH1 (SHIELD), J1.SH2 (SHIELD__1)
- net RS_A: now reaches U4.6 (A)
- net RS_A: now also J1.1
- net RS_B: now reaches U4.7 (B)
- net RS_B: now also J1.2
- net +BATT: now reaches U2.1 (VIN)
- net +BATT: now also U2.3 (CE), C2.1
- net DIO3: now reaches U1.11 (DIO3)
- net DIO1: now reaches U1.15 (DIO1)
- net BUSY: now reaches U1.16 (BUSY)
- net MISO: now reaches U1.2 (MISO)
- net MOSI: now reaches U1.3 (MOSI)
- net SCK: now reaches U1.4 (SCK)
- net CS_1: now reaches U1.5 (NSS)
- net NRESET: now reaches U1.6 (NRESET)
- net at U1.9 (ANT): now also AE1.1 (A)
- new net: J1.10, R1.2
- new net: J1.12, R2.2
- new net: J1.3, J1.6
- new net +6V: J1.4, J1.5
- new net LED_GRN: R1.1
- new net LED_YLW: R2.1
- no-connect marks 0 -> 4
Other:
- moved on the sheet: U1, U2, U4
