File: hardware/satellite-board/satellite-board.kicad_pcb (KiCad board)
At the start: 2 copper layers, 6.5 x 0.7 mm, 27 parts, among them J1 MTJ-88ARX1-FSM-LG, J2 B2B-PH-K-S, Q1 2N7002, U1 LORA1262-915TCXO, U2 XC6220B331MR, U3 ESP32-C6-DEVKITC-1-N8, U4 MAX3485

Commit message: Layout started
Parts:
- J1, U6: moved to B.Cu
- moved C4 84.5 mm to (90.6, 55.9)
- moved C5 84.5 mm to (90.6, 57.9)
- moved C6 84.5 mm to (90.6, 59.8)
- moved C8 84.5 mm to (90.6, 61.8)
- moved D1 84.5 mm to (99.3, 62.6)
- moved U4 84.5 mm to (96.9, 71.8)
- moved C2 84.5 mm to (89.0, 96.0)
- moved C3 84.5 mm to (89.0, 98.5)
- moved CN1 84.5 mm to (96.9, 78.5)
- moved J2 84.5 mm to (92.1, 51.1)
- moved Q1 84.5 mm to (94.5, 65.1)
- moved R1 84.5 mm to (89.0, 101.1)
- moved R2 84.5 mm to (89.0, 103.6)
- moved R3 84.5 mm to (89.0, 106.1)
- moved R5 84.5 mm to (99.4, 59.7)
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Other:
- board size 6.5 x 0.7 mm -> 65 x 56 mm

Commit message: Satelite Board Started
Parts:
- removed D1: ~, Diode_SMD:D_SOD-323F
- added R7: 4.7k, Resistor_SMD:R_0402_1005Metric, F.Cu at (180.8, 93.5)
- Q1: value 2N7002 -> MMBT3904
- R6: value 100k -> 47k
- U6: moved to F.Cu
- moved CN1 129.2 mm to (225.4, 65.2), turned to 90 degrees
- moved R3 126.4 mm to (191.4, 32.0)
- moved C3 117.4 mm to (204.0, 75.4)
- moved C4 114.7 mm to (203.3, 76.8)
- moved J2 104.6 mm to (186.6, 96.0)
- moved R1 98.6 mm to (174.8, 52.6), turned to 90 degrees
- moved C2 96.7 mm to (185.6, 92.9)
- moved C1 96.6 mm to (185.7, 86.8)
- moved U2 95.7 mm to (185.7, 90.0), turned to 90 degrees
- moved R2 95.2 mm to (174.8, 62.4), turned to -90 degrees
- moved Q1 93.5 mm to (182.1, 97.6)
- moved R6 88.0 mm to (181.3, 95.2)
- moved C5 73.0 mm to (161.7, 74.0)
- moved C6 72.3 mm to (161.7, 72.8)
- moved C9 72.2 mm to (157.8, 49.8), turned to 180 degrees
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Connections:
- Q1 pad 1: GPS_RESET -> Net-(Q1-B)
- R6 pad 1: GPS_RESET -> Net-(Q1-B)
- U3 pad J1_13: RS_EN -> BUSY
- U3 pad J3_5: BUSY -> RS_EN
Routing:
- net GND: track 0.00 -> 56.2 mm, vias 0 -> 153
- net +3V3: track 0.00 -> 51.7 mm
- net Net-(Q1-C): track 0.00 -> 19.2 mm
- net RS_EN: track 0.00 -> 18.6 mm, vias 0 -> 1
- net RS_TX: track 0.00 -> 15.7 mm, vias 0 -> 1
- net NRESET: track 0.00 -> 13.3 mm
- net Net-(J1-Pad3): track 0.00 -> 13.0 mm
- net GPS_RX: track 0.00 -> 12.4 mm
- net +BATT: track 0.00 -> 11.8 mm, vias 0 -> 1
- net CS_1: track 0.00 -> 11.2 mm
- net RS_B: track 0.00 -> 10.7 mm
- net GPS_TX: track 0.00 -> 10.3 mm, vias 0 -> 1
- net SCK: track 0.00 -> 8.48 mm
- net RS_A: track 0.00 -> 7.53 mm
- net MOSI: track 0.00 -> 6.29 mm
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- added copper zone on B.Cu, net GND
- added copper zone on F.Cu, net GND

Commit message: Updates to Sat
Parts:
- moved R4 82.5 mm to (177.0, 63.1), turned to -90 degrees
- moved USB1 40.9 mm to (182.9, 52.6)
- moved CN1 40.5 mm to (185.0, 61.8)
- moved R3 30.8 mm to (177.0, 59.2), turned to -90 degrees
- moved R1 1.65 mm to (174.8, 51.0), turned to -90 degrees
Connections:
- U3 pad J1_10: LED_GRN -> RJ45_SNS
- U3 pad J1_11: LED_YLW -> DIO1
- U3 pad J3_6: DIO1 -> LED_YLW
- U3 pad J3_7: RJ45_SNS -> LED_GRN
Routing:
- net VBUS: track 2.20 -> 25.2 mm
- net LED_YLW: track 0.00 -> 18.1 mm, vias 0 -> 1
- net RJ45_SNS: track 0.00 -> 9.63 mm
- net LED_GRN: track 0.00 -> 5.63 mm
Changed lines of the file:
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@@
 	(footprint "Resistor_SMD:R_1206_3216Metric"
 		(layer "F.Cu")
-		(at 94.805 56.565)
+		(at 177 63.1375 -90)
 		(descr "Resistor SMD 1206 (3216 Metric), square (rectangular) end terminal, IPC-7351 nominal, (Body size source: IPC-SM-782 page 72, https://www.pcb-3d.com/wordpress/wp-content/uploads/ipc-sm-782a_amendment_1_and_2.pdf), generated with kicad-footprint-generator")
 		(tags "resistor")
 		(property "Reference" "R4"
-			(at 0 -1.83 0)
+			(at 0 -1.83 90)
 			(layer "F.SilkS")
 			(effects
@@
 		)
 		(property "Value" "4.7k"
-			(at 0 1.83 0)
+			(at 0 1.83 90)
 			(layer "F.Fab")
+			(hide yes)
 			(effects
 				(font
@@
 		)
 		(property "Datasheet" "~"
-			(at 0 0 0)
+			(at 0 0 90)
 			(layer "F.Fab")
 			(hide yes)
@@
 		)
 		(property "Description" "Resistor"
-			(at 0 0 0)
+			(at 0 0 90)
 			(layer "F.Fab")
 			(hide yes)
@@
 		)
 		(property "LCSC" "C17936"
-			(at 0 0 0)
+			(at 0 0 270)
 			(unlocked yes)
 			(layer "F.Fab")
@@
 		(attr smd)
 		(fp_line
-			(start -0.727064 -0.91)
-			(end 0.727064 -0.91)
+			(start -0.727064 0.91)
+			(end 0.727064 0.91)
 			(stroke
 				(width 0.12)
@@
 		)
 		(fp_line
-			(start -0.727064 0.91)
-			(end 0.727064 0.91)
+			(start -0.727064 -0.91)
+			(end 0.727064 -0.91)
 			(stroke
 				(width 0.12)
@@
 		)
 		(fp_text user "${REFERENCE}"
-			(at 0 0 0)
+			(at 0 0 90)
 			(layer "F.Fab")
 			(effects
@@
 		)
 		(pad "1" smd roundrect
-			(at -1.4625 0)
+			(at -1.4625 0 270)
 			(size 1.125 1.75)
 			(layers "F.Cu" "F.Mask" "F.Paste")
@@
 		)
 		(pad "2" smd roundrect
-			(at 1.4625 0)
+			(at 1.4625 0 270)
 			(size 1.125 1.75)
 			(layers "F.Cu" "F.Mask" "F.Paste")
@@
 			(layers "*.Cu" "*.Mask")
 			(remove_unused_layers no)
-			(net 13 "LED_GRN")
+			(net 15 "RJ45_SNS")
 			(pinfunction "GPIO10")
 			(pintype "bidirectional")
@@
 			(layers "*.Cu" "*.Mask")
 			(remove_unused_layers no)
-			(net 14 "LED_YLW")
+			(net 25 "DIO1")
 			(pinfunction "GPIO11")
 			(pintype "bidirectional")
@@
 			(layers "*.Cu" "*.Mask")
 			(remove_unused_layers no)
-			(net 25 "DIO1")
+			(net 14 "LED_YLW")
 			(pinfunction "GPIO22")
 			(pintype "bidirectional")
@@
 			(layers "*.Cu" "*.Mask")
 			(remove_unused_layers no)
-			(net 15 "RJ45_SNS")
+			(net 13 "LED_GRN")
 			(pinfunction "GPIO21")
 			(pintype "bidirectional")
@@
 	(footprint "Resistor_SMD:R_0603_1608Metric"
 		(layer "F.Cu")
-		(at 191.4 32)
+		(at 177 59.175 -90)
 		(descr "Resistor SMD 0603 (1608 Metric), square (rectangular) end terminal, IPC-7351 nominal, (Body size source: IPC-SM-782 page 72, https://www.pcb-3d.com/wordpress/wp-content/uploads/ipc-sm-782a_amendment_1_and_2.pdf), generated with kicad-footprint-generator")
 		(tags "resistor")
 		(property "Reference" "R3"
-			(at 0 -1.43 0)
+			(at 0 -1.43 90)
 			(layer "F.SilkS")
 			(effects
@@
 		)
 		(property "Value" "15K"
-			(at 0 1.43 0)
+			(at 0 1.43 90)
 			(layer "F.Fab")
+			(hide yes)
 			(effects
 				(font
@@
 		)
 		(property "Datasheet" "~"
-			(at 0 0 0)
+			(at 0 0 90)
 			(layer "F.Fab")
 			(hide yes)
@@
 		)
 		(property "Description" "Resistor"
-			(at 0 0 0)
+			(at 0 0 90)
 			(layer "F.Fab")
 			(hide yes)
@@
 		)
 		(property "LCSC" "C22809"
-			(at 0 0 0)
+			(at 0 0 270)
 			(unlocked yes)
 			(layer "F.Fab")
@@
 		(attr smd)
 		(fp_line
-			(start -0.237258 -0.5225)
-			(end 0.237258 -0.5225)
+			(start -0.237258 0.5225)
+			(end 0.237258 0.5225)
 			(stroke
 				(width 0.12)
@@
 		)
 		(fp_line
-			(start -0.237258 0.5225)
-			(end 0.237258 0.5225)
+			(start -0.237258 -0.5225)
+			(end 0.237258 -0.5225)
 			(stroke
 				(width 0.12)
@@
 		)
 		(fp_text user "${REFERENCE}"
-			(at 0 0 0)
+			(at 0 0 90)
 			(layer "F.Fab")
 			(effects
@@
 		)
 		(pad "1" smd roundrect
-			(at -0.825 0)
+			(at -0.825 0 270)
 			(size 0.8 0.95)
 			(layers "F.Cu" "F.Mask" "F.Paste")
@@
 		)
 		(pad "2" smd roundrect
-			(at 0.825 0)
+			(at 0.825 0 270)
 			(size 0.8 0.95)
 			(layers "F.Cu" "F.Mask" "F.Paste")
@@
 	(footprint "library:CONN-SMD_4P-P1.00_XY-SM04B-SRSS-TB"
 		(layer "F.Cu")
-		(at 225.4 65.2 90)
+		(at 185 61.8 90)
 		(property "Reference" "CN1"
 			(at 0 -3.775 90)
@@
 	(footprint "Resistor_SMD:R_0603_1608Metric"
 		(layer "F.Cu")
-		(at 174.8 52.625 90)
+		(at 174.8 50.975 -90)
 		(descr "Resistor SMD 0603 (1608 Metric), square (rectangular) end terminal, IPC-7351 nominal, (Body size source: IPC-SM-782 page 72, https://www.pcb-3d.com/wordpress/wp-content/uploads/ipc-sm-782a_amendment_1_and_2.pdf), generated with kicad-footprint-generator")
 		(tags "resistor")
 		(property "Reference" "R1"
-			(at 2.2 0 180)
+			(at 2.2 0 0)
 			(layer "F.SilkS")
 			(effects
@@
 		)
 		(property "LCSC" "C22808"
-			(at 0 0 90)
+			(at 0 0 270)
 			(unlocked yes)
 			(layer "F.Fab")
@@
 		(attr smd)
 		(fp_line
-			(start -0.237258 -0.5225)
-			(end 0.237258 -0.5225)
+			(start -0.237258 0.5225)
+			(end 0.237258 0.5225)
 			(stroke
 				(width 0.12)
@@
 		)
 		(fp_line
-			(start -0.237258 0.5225)
-			(end 0.237258 0.5225)
+			(start -0.237258 -0.5225)
+			(end 0.237258 -0.5225)
 			(stroke
 				(width 0.12)
@@
 		)
 		(pad "1" smd roundrect
-			(at -0.825 0 90)
+			(at -0.825 0 270)
 			(size 0.8 0.95)
 			(layers "F.Cu" "F.Mask" "F.Paste")
@@
 		)
 		(pad "2" smd roundrect
-			(at 0.825 0 90)
+			(at 0.825 0 270)
 			(size 0.8 0.95)
 			(layers "F.Cu" "F.Mask" "F.Paste")
@@
 	(footprint "Library:USB-C-SMD_TYPE-C-6PIN-2MD-073"
 		(layer "F.Cu")
-		(at 223.74925 50.2 90)
+		(at 182.94925 52.6 90)
 		(property "Reference" "USB1"
-			(at 0 -3.9 90)
+			(at 0 0 90)
 			(layer "F.SilkS")
 			(effects
@@
 	)
 	(segment
-		(start 172.54 51.83)
-		(end 174.77 51.83)
+		(start 174.77 51.83)
+		(end 174.8 51.8)
 		(width 0.35)
 		(layer "F.Cu")
@@
 	)
 	(segment
-		(start 174.77 51.83)
-		(end 174.8 51.8)
+		(start 172.54 51.83)
+		(end 174.77 51.83)
 		(width 0.35)
 		(layer "F.Cu")
@@
 	)
 	(segment
+		(start 179.2 54.6)
+		(end 179.6 55)
+		(width 0.7)
+		(layer "F.Cu")
+		(net 11)
+	)
+	(segment
 		(start 166.29 56.91)
 		(end 166.8 56.4)
@@
 	)
 	(segment
+		(start 179.2 50.6)
+		(end 179.2 52.4)
+		(width 0.7)
+		(layer "F.Cu")
+		(net 11)
+	)
+	(segment
+		(start 179.6 50.2)
+		(end 179.2 50.6)
+		(width 0.7)
+		(layer "F.Cu")
+		(net 11)
+	)
+	(segment
+		(start 175.71 55.89)
+		(end 179.2 52.4)
+		(width 0.7)
+		(layer "F.Cu")
+		(net 11)
+	)
+	(segment
 		(start 167.21 56.4)
 		(end 167.72 55.89)
@@
 	)
 	(segment
+		(start 179.2 52.4)
+		(end 179.2 54.6)
+		(width 0.7)
+		(layer "F.Cu")
+		(net 11)
+	)
+	(segment
+		(start 177 57.18)
+		(end 175.71 55.89)
+		(width 0.7)
+		(layer "F.Cu")
+		(net 11)
+	)
+	(segment
+		(start 180.57425 50.2)
+		(end 179.6 50.2)
+		(width 0.5)
+		(layer "F.Cu")
+		(net 11)
+	)
+	(segment
+		(start 179.6 55)
+		(end 180.57425 55)
+		(width 0.5)
+		(layer "F.Cu")
+		(net 11)
+	)
+	(segment
+		(start 167.72 55.89)
+		(end 175.71 55.89)
+		(width 1)
+		(layer "F.Cu")
+		(net 11)
+	)
+	(segment
+		(start 177 58.35)
+		(end 177 57.18)
+		(width 0.7)
+		(layer "F.Cu")
+		(net 11)
+	)
+	(segment
 		(start 165.94 56.91)
 		(end 166.29 56.91)
@@
 	)
 	(segment
+		(start 174.8 50.15)
+		(end 174.8 46.055)
+		(width 0.35)
+		(layer "F.Cu")
+		(net 13)
+	)
+	(segment
+		(start 174.8 46.055)
+		(end 173.715 44.97)
+		(width 0.35)
+		(layer "F.Cu")
+		(net 13)
+	)
+	(segment
+		(start 174.8 61.6)
+		(end 174.8 57.4)
+		(width 0.35)
+		(layer "F.Cu")
+		(net 14)
+	)
+	(via
+		(at 174.8 57.4)
+		(size 0.6)
+		(drill 0.3)
+		(layers "F.Cu" "B.Cu")
+		(net 14)
+	)
+	(segment
+		(start 172.405 46.205)
+		(end 172.405 46.2)
+		(width 0.35)
+		(layer "B.Cu")
+		(net 14)
+	)
+	(segment
+		(start 174.8 48.6)
+		(end 172.405 46.205)
+		(width 0.35)
+		(layer "B.Cu")
+		(net 14)
+	)
+	(segment
+		(start 174.8 57.4)
+		(end 174.8 48.6)
+		(width 0.35)
+		(layer "B.Cu")
+		(net 14)
+	)
+	(segment
+		(start 172.405 46.2)
+		(end 171.175 44.97)
+		(width 0.35)
+		(layer "B.Cu")
+		(net 14)
+	)
+	(segment
+		(start 181.335 66.01)
+		(end 177 61.675)
+		(width 0.25)
+		(layer "F.Cu")
+		(net 15)
+	)
+	(segment
+		(start 181.335 67.83)
+		(end 181.335 66.01)
+		(width 0.25)
+		(layer "F.Cu")
+		(net 15)
+	)
+	(segment
+		(start 177 60)
+		(end 177 61.675)
+		(width 0.7)
+		(layer "F.Cu")
+		(net 15)
+	)
+	(segment

Commit message: Branch updates
Connections:
- U3 pad J1_11: DIO1 -> CS_1
- U3 pad J1_8: CS_1 -> GPS_RESET
- U3 pad J3_8: GPS_RESET -> DIO1
Routing:
- net +3V3: track 51.7 -> 132.5 mm
- net SCK: track 8.48 -> 62.1 mm, vias 0 -> 1
- net DIO1: track 0.00 -> 49.3 mm, vias 0 -> 3
- net MOSI: track 6.29 -> 54.6 mm, vias 0 -> 1
- net NRESET: track 13.3 -> 59.3 mm, vias 0 -> 1
- net CS_1: track 11.2 -> 47.4 mm, vias 0 -> 1
- net MISO: track 4.11 -> 37.1 mm
- net GPS_RESET: track 0.00 -> 28.5 mm, vias 0 -> 1
- net SDA: track 0.00 -> 18.4 mm
- net SCL: track 0.00 -> 17.5 mm
- net BUSY: track 0.00 -> 14.3 mm
- net GND: track 56.2 -> 62.7 mm, vias 153 -> 152
- net Net-(J1-Pad3): track 13.0 -> 13.7 mm
Other:
- board text added: "Designed by Michael Danley"
- board text added: "Project ORCA - SATELLITE"
- board text added: "Sensor Data Transmit Hub"

Commit message: Prepared for production
Parts:
- moved C1 79.9 mm to (106.8, 73.9)
- moved C2 79.9 mm to (106.7, 80.0)
- moved C3 79.9 mm to (125.1, 62.5)
- moved C5 79.9 mm to (82.8, 61.1)
- moved C6 79.9 mm to (82.8, 59.9)
- moved C8 79.9 mm to (79.8, 38.7)
- moved CN1 79.9 mm to (106.1, 48.9)
- moved J1 79.9 mm to (84.5, 43.5)
- moved Q1 79.9 mm to (103.2, 84.7)
- moved R1 79.9 mm to (95.9, 38.1)
- moved R2 79.9 mm to (95.9, 49.5)
- moved R3 79.9 mm to (98.1, 46.3)
- moved R4 79.9 mm to (98.1, 50.2)
- moved R7 79.9 mm to (101.9, 80.6)
- moved U2 79.9 mm to (106.8, 77.1)
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Routing:
- net GND: vias 152 -> 204
